File: pcb/traction-control/output.kicad_sch (KiCad schematic)
At the start: 4 parts, among them Q5 Q_Dual_PMOS_S1G1S2G2D2D2D1D1, Q6 AO3400A

Commit message: Revision and production files
Parts:
- R11: renamed from R12; LCSC (none) -> C25900
- renumbered D4 to D3
Changed lines of the file:
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@@
 		(dnp no)
 		(fields_autoplaced yes)
-		(property "Reference" "#PWR044"
+		(property "Reference" "#PWR047"
 			(at 74.93 50.8 0)
 			(effects
@@
 			(project "traction-control"
 				(path "/eb07aa05-a882-45b0-b9de-bffe5728f99f/38342423-5a8c-4a47-a7cd-f2e71952ef73"
-					(reference "#PWR044")
-					(unit 1)
-				)
-				(path "/eb07aa05-a882-45b0-b9de-bffe5728f99f/96f55cd2-4032-4864-9209-b13ab493c175"
-					(reference "#PWR038")
+					(reference "#PWR047")
+					(unit 1)
+				)
+				(path "/eb07aa05-a882-45b0-b9de-bffe5728f99f/96f55cd2-4032-4864-9209-b13ab493c175"
+					(reference "#PWR042")
 					(unit 1)
 				)
@@
 		(dnp no)
 		(fields_autoplaced yes)
-		(property "Reference" "#PWR047"
+		(property "Reference" "#PWR050"
 			(at 52.07 81.28 0)
 			(effects
@@
 			(project "traction-control"
 				(path "/eb07aa05-a882-45b0-b9de-bffe5728f99f/38342423-5a8c-4a47-a7cd-f2e71952ef73"
-					(reference "#PWR047")
-					(unit 1)
-				)
-				(path "/eb07aa05-a882-45b0-b9de-bffe5728f99f/96f55cd2-4032-4864-9209-b13ab493c175"
-					(reference "#PWR041")
+					(reference "#PWR050")
+					(unit 1)
+				)
+				(path "/eb07aa05-a882-45b0-b9de-bffe5728f99f/96f55cd2-4032-4864-9209-b13ab493c175"
+					(reference "#PWR045")
 					(unit 1)
 				)
@@
 		(dnp no)
 		(fields_autoplaced yes)
-		(property "Reference" "#PWR046"
+		(property "Reference" "#PWR049"
 			(at 102.87 53.34 0)
 			(effects
@@
 			(project "traction-control"
 				(path "/eb07aa05-a882-45b0-b9de-bffe5728f99f/38342423-5a8c-4a47-a7cd-f2e71952ef73"
-					(reference "#PWR046")
-					(unit 1)
-				)
-				(path "/eb07aa05-a882-45b0-b9de-bffe5728f99f/96f55cd2-4032-4864-9209-b13ab493c175"
-					(reference "#PWR040")
+					(reference "#PWR049")
+					(unit 1)
+				)
+				(path "/eb07aa05-a882-45b0-b9de-bffe5728f99f/96f55cd2-4032-4864-9209-b13ab493c175"
+					(reference "#PWR044")
 					(unit 1)
 				)
@@
 		(dnp no)
 		(fields_autoplaced yes)
-		(property "Reference" "#PWR045"
+		(property "Reference" "#PWR048"
 			(at 95.25 50.8 0)
 			(effects
@@
 			(project "traction-control"
 				(path "/eb07aa05-a882-45b0-b9de-bffe5728f99f/38342423-5a8c-4a47-a7cd-f2e71952ef73"
-					(reference "#PWR045")
-					(unit 1)
-				)
-				(path "/eb07aa05-a882-45b0-b9de-bffe5728f99f/96f55cd2-4032-4864-9209-b13ab493c175"
-					(reference "#PWR039")
+					(reference "#PWR048")
+					(unit 1)
+				)
+				(path "/eb07aa05-a882-45b0-b9de-bffe5728f99f/96f55cd2-4032-4864-9209-b13ab493c175"
+					(reference "#PWR043")
 					(unit 1)
 				)
@@
 		(dnp no)
 		(fields_autoplaced yes)
-		(property "Reference" "D4"
+		(property "Reference" "D3"
 			(at 105.41 54.2924 90)
 			(effects
@@
 			(project "traction-control"
 				(path "/eb07aa05-a882-45b0-b9de-bffe5728f99f/38342423-5a8c-4a47-a7cd-f2e71952ef73"
-					(reference "D4")
+					(reference "D3")
 					(unit 1)
 				)
@@
 		(dnp no)
 		(fields_autoplaced yes)
-		(property "Reference" "#PWR043"
+		(property "Reference" "#PWR046"
 			(at 52.07 50.8 0)
 			(effects
@@
 			(project "traction-control"
 				(path "/eb07aa05-a882-45b0-b9de-bffe5728f99f/38342423-5a8c-4a47-a7cd-f2e71952ef73"
-					(reference "#PWR043")
-					(unit 1)
-				)
-				(path "/eb07aa05-a882-45b0-b9de-bffe5728f99f/96f55cd2-4032-4864-9209-b13ab493c175"
-					(reference "#PWR037")
+					(reference "#PWR046")
+					(unit 1)
+				)
+				(path "/eb07aa05-a882-45b0-b9de-bffe5728f99f/96f55cd2-4032-4864-9209-b13ab493c175"
+					(reference "#PWR041")
 					(unit 1)
 				)
@@
 		(dnp no)
 		(fields_autoplaced yes)
-		(property "Reference" "R12"
+		(property "Reference" "R11"
 			(at 54.61 52.0699 0)
 			(effects
@@
 			)
 		)
+		(property "LCSC" "C25900"
+			(at 52.07 53.34 0)
+			(effects
+				(font
+					(size 1.27 1.27)
+				)
+				(hide yes)
+			)
+		)
 		(pin "2"
 		)
@@
 			(project "traction-control"
 				(path "/eb07aa05-a882-45b0-b9de-bffe5728f99f/38342423-5a8c-4a47-a7cd-f2e71952ef73"
-					(reference "R12")
-					(unit 1)
-				)
+					(reference "R11")
+					(unit 1)
+				)

Commit message: Save
Parts:
- Q6: LCSC (none) -> C20917
Changed lines of the file:
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@@
+			)
+		)
+		(property "LCSC" "C20917"
+			(at 49.53 67.31 0)
+			(effects
+				(font
+					(size 1.27 1.27)
+				)
+				(hide yes)
 			)
 		)

Commit message: Make production files
Parts:
- Q5: value Q_Dual_PMOS_S1G1S2G2D2D2D1D1 -> DMP4025LSD-VB
Changed lines of the file:
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@@
 			)
 		)
-		(property "Value" "Q_Dual_PMOS_S1G1S2G2D2D2D1D1"
+		(property "Value" "DMP4025LSD-VB"
 			(at 99.06 53.3401 0)
 			(effects
@@
 		(dnp no)
 		(property "Reference" "Q5"
-			(at 76.454 51.054 0)
-			(effects
-				(font
-					(size 1.27 1.27)
-				)
-				(justify left)
-			)
-		)
-		(property "Value" "Q_Dual_PMOS_S1G1S2G2D2D2D1D1"
-			(at 78.74 53.3401 0)
-			(effects
-				(font
-					(size 1.27 1.27)
-				)
-				(justify left)
-				(hide yes)
-			)
-		)
+			(at 68.326 50.546 0)
+			(effects
+				(font
+					(size 1.27 1.27)
+				)
+				(justify left)
+			)
+		)
+		(property "Value" "DMP4025LSD-VB"
+			(at 76.454 48.006 0)
+			(effects
+				(font
+					(size 1.27 1.27)
+				)
+				(justify left)
+			)
+		)
