File: pcb/traction-control/sensor.kicad_sch (KiCad schematic)
At the start: 3 parts

Commit message: Save
Parts:
- renumbered R17 to R12, R19 to R14
Changed lines of the file:
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@@
 		(dnp no)
 		(fields_autoplaced yes)
-		(property "Reference" "#PWR056"
+		(property "Reference" "#PWR052"
 			(at 53.34 95.25 0)
 			(effects
@@
 		(dnp no)
 		(fields_autoplaced yes)
-		(property "Reference" "R19"
+		(property "Reference" "R14"
 			(at 55.88 81.2799 0)
 			(effects
@@
 		(dnp no)
 		(fields_autoplaced yes)
-		(property "Reference" "R17"
+		(property "Reference" "R12"
 			(at 55.88 55.8799 0)
 			(effects
@@
 		(dnp no)
 		(fields_autoplaced yes)
-		(property "Reference" "#PWR055"
+		(property "Reference" "#PWR051"
 			(at 53.34 54.61 0)
 			(effects

Commit message: Make production files
Parts:
- R12: LCSC (none) -> C4410
- R13: LCSC (none) -> C25768
- R14: value 4k7 -> 5k1; LCSC C25900 -> C25905
Changed lines of the file:
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@@
 			)
 		)
-		(property "Value" "4k7"
+		(property "Value" "5k1"
 			(at 55.88 83.8199 0)
 			(effects
@@
 			)
 		)
-		(property "LCSC" "C25900"
+		(property "LCSC" "C25905"
 			(at 53.34 82.55 0)
 			(effects
@@
 			)
 		)
+		(property "LCSC" "C4410"
+			(at 53.34 57.15 0)
+			(effects
+				(font
+					(size 1.27 1.27)
+				)
+				(hide yes)
+			)
+		)
 		(pin "1"
 		)
@@
 			(at 53.34 69.85 0)
 			(effects
+				(font
+					(size 1.27 1.27)
+				)
+				(hide yes)
+			)
+		)
+		(property "LCSC" "C25768"
+			(at 53.34 69.85 0)
+			(effects
