File: pcb/traction-control/tac.kicad_sch (KiCad schematic)
At the start: 3 parts

Commit message: Revision and production files
Parts:
- removed R13: 22k, Resistor_SMD:R_0402_1005Metric, symbol Device:R
- removed R17: 1k, Resistor_SMD:R_1206_3216Metric, symbol Device:R
- removed R19: 4k7, Resistor_SMD:R_0402_1005Metric, symbol Device:R
- added D4: MM1Z3V3, Diode_SMD:D_SOD-123, symbol Device:D_Zener
- added R15: 18k, Resistor_SMD:R_1206_3216Metric, symbol Device:R
- added R16: 2k2, Resistor_SMD:R_1206_3216Metric, symbol Device:R
Connections:
- net GND: now also D4.2 (A), R16.2
- net OUT: now also D4.1 (K), R15.2, R16.1
- net SNS: now also R15.1

Commit message: Make production files
Parts:
- removed D4: MM1Z3V3, Diode_SMD:D_SOD-123, symbol Device:D_Zener
- removed R15: 18k, Resistor_SMD:R_1206_3216Metric, symbol Device:R
- removed R16: 2k2, Resistor_SMD:R_1206_3216Metric, symbol Device:R
- added D5: SS54, Diode_SMD:D_SMA, symbol Device:D_Schottky
- added R20: 10k, Resistor_SMD:R_0402_1005Metric, symbol Device:R
- added R21: 5k1, Resistor_SMD:R_0402_1005Metric, symbol Device:R
- added R22: 47k, Resistor_SMD:R_0402_1005Metric, symbol Device:R
- added R23: 12k, Resistor_SMD:R_0402_1005Metric, symbol Device:R
Connections:
- net GND: now also R21.2, R23.2
- net OUT: now also R22.2, R23.1
- net SNS: now also R20.1
- new net +12V: D5.1 (K)
- new net PROT: D5.2 (A), R20.2, R21.1, R22.1
