File: pcb/traction-control/traction-control.kicad_pcb (KiCad board)
At the start: 4 copper layers, 43.6 x 43.6 mm, 78 parts, among them J1 Conn_01x05_Socket, J2 Conn_01x04_Pin, J3 Screw_Terminal_01x06, J4 Conn_01x04_Pin, J5 Conn_ARM_SWD_TagConnect_TC203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, Q1 AO3400A, Q10 AO3400A, Q2 AO3401A, Q3 Q_Dual_PMOS_S1G1S2G2D2D2D1D1, Q4 AO3400A, Q5 Q_Dual_PMOS_S1G1S2G2D2D2D1D1, Q6 AO3400A, Q7 AO3401A, Q8 AO3400A, Q9 AO3400A, SW1 SW_Push, SW2 SW_Push, SW3 SW_Push, SW4 SW_Push, U1 AT24CS32-SSHM, U2 STM32F103C8Tx, U3 AMS1117-3.3, U4 TPS5430DDA, U5 LM393, Y1 16MHz

Commit message: Revision and production files
Parts:
- removed the C18 at (95.3, 75.8)
- removed C19, C21: 1n, Capacitor_SMD:C_0402_1005Metric
- removed C20: 150p, Capacitor_SMD:C_0402_1005Metric
- removed D6: SS54, Diode_SMD:D_SMA
- removed Q10, Q8, Q9: AO3400A, Package_TO_SOT_SMD:SOT-23
- removed Q7: AO3401A, Package_TO_SOT_SMD:SOT-23
- removed the R17 at (93.3, 75.8)
- removed the R18 at (103.6, 77.1)
- removed the R19 at (109.7, 76.8)
- removed R20: 5k, Resistor_SMD:R_0402_1005Metric
- removed R21: 100k, Resistor_SMD:R_0402_1005Metric
- removed U5: LM393, Package_SO:SOIC-8_3.9x4.9mm_P1.27mm
- added D4: MM1Z3V3, Diode_SMD:D_SOD-123, F.Cu at (103.9, 75.8)
- added G1: LOGO, LOGO, B.Cu at (93.9, 86.4)
- added JP1: SolderJumper_3_Open, Jumper:SolderJumper-3_P1.3mm_Open_RoundedPad1.0x1.5mm, B.Cu at (109.9, 89.1)
- added R12: 1k, Resistor_SMD:R_1206_3216Metric, F.Cu at (109.7, 77.0)
- added R13: 22k, Resistor_SMD:R_0402_1005Metric, F.Cu at (102.1, 78.4)
- R15: value 1k -> 18k
- R16: value 15k -> 2k2; footprint Resistor_SMD:R_0402_1005Metric -> Resistor_SMD:R_1206_3216Metric
- R18: renamed from R11; value 10k -> 22k
- moved Y1 19.5 mm to (98.1, 76.4), turned to -90 degrees
- moved C8 18.9 mm to (98.9, 73.7), turned to 180 degrees
- moved C2 18.1 mm to (93.3, 80.0), turned to 180 degrees
- moved C9 17.3 mm to (95.9, 77.5), turned to 90 degrees
- moved R4 16.9 mm to (91.4, 80.0), turned to 180 degrees
- moved R5 15.1 mm to (95.9, 75.6), turned to 90 degrees
- moved C7 14.9 mm to (96.9, 72.8), turned to 90 degrees
- moved C5 13.8 mm to (84.3, 77.1), turned to 90 degrees
- moved C3 13.1 mm to (95.9, 72.8), turned to -90 degrees
- moved Q1 10.3 mm to (84.1, 63.9), turned to -90 degrees
- moved R16 9.96 mm to (107.4, 77.0), turned to 90 degrees
- moved R8 8.44 mm to (87.1, 66.3)
- moved R9 7.94 mm to (89.9, 66.3)
- moved C4 6.28 mm to (87.1, 68.4), turned to 0 degrees
- moved U2 5.85 mm to (90.0, 74.2), turned to 180 degrees
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- renumbered C24 to C17, C17 to C18, D8 to D1, D4 to D3, J5 to J3, J3 to J4, J4 to J5, R12 to R11, R13 to R17, R22 to R19
Connections:
- J4 pad 5: /SNS1 -> /SNS3
- J4 pad 6: /SNS2 -> Net-(J4-Pin_6)
- R14 pad 1: +12V -> /SIG3
- R14 pad 2: Net-(Q7-G) -> GND
- R15 pad 1: Net-(Q7-D) -> /SNS1
- R15 pad 2: /SNS1 -> /SIG1
- R16 pad 1: +12V -> /SIG1
- R16 pad 2: Net-(U5B--) -> GND
- R18 pad 2: Net-(Q10-G) -> /SIG2
- R19 pad 1: Net-(Q10-G) -> /SIG2
- U2 pad 12: /GPS_TX -> unconnected-(U2-PA2-Pad12)
- U2 pad 13: /GPS_RX -> /SIG2
- U2 pad 14: unconnected-(U2-PA4-Pad14) -> /SIG3
- U2 pad 15: unconnected-(U2-PA5-Pad15) -> /SIG1
- U2 pad 16: unconnected-(U2-PA6-Pad16) -> /DRV2
- U2 pad 17: unconnected-(U2-PA7-Pad17) -> /DRV1
- U2 pad 21: /SCLE -> /SCLD
- U2 pad 22: /SDAE -> /SDAD
- U2 pad 25: unconnected-(U2-PB12-Pad25) -> /PGPS
- U2 pad 3: unconnected-(U2-PC14-Pad3) -> /BTN3
- U2 pad 30: unconnected-(U2-PA9-Pad30) -> /GPS_TX
- U2 pad 31: unconnected-(U2-PA10-Pad31) -> /GPS_RX
- U2 pad 4: unconnected-(U2-PC15-Pad4) -> /BTN4
- U2 pad 42: /SCLD -> /SCLE
- U2 pad 43: /SDAD -> /SDAE
- U2 pad 45: unconnected-(U2-PB8-Pad45) -> /BTN1
- U2 pad 46: unconnected-(U2-PB9-Pad46) -> /BTN2
Routing:
- net +12V: track 19.4 -> 65.7 mm, vias 0 -> 10
- net /SWO: track 1.74 -> 30.7 mm, vias 0 -> 1
- net /BTN4: track 0.00 -> 27.9 mm, vias 0 -> 3
- net /SIG2: track 0.00 -> 26.2 mm
- net /SIG1: track 0.00 -> 23.7 mm
- net /SIG3: track 0.00 -> 19.2 mm
- net /SNS3: track 0.00 -> 17.7 mm, vias 0 -> 1
- net /BTN1: track 7.95 -> 24.0 mm, vias 0 -> 2
- net /SWCLK: track 17.5 -> 33.0 mm
- net /SWDIO: track 13.0 -> 28.4 mm
- net /DRV1: track 0.00 -> 13.3 mm
- net +3V3: track 73.0 -> 60.6 mm, vias 8 -> 10
- net /BTN3: track 7.95 -> 19.1 mm, vias 0 -> 2
- net /DRV2: track 0.00 -> 11.1 mm
- net /BTN2: track 7.95 -> 17.8 mm, vias 0 -> 2
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- added copper zone on F.Cu, net +12V
- added copper zone on In2.Cu, net +12V
- added copper zone on In2.Cu, net +3V3
- added copper zone on F.Cu, net /OUT1
- added copper zone on F.Cu, net /OUT2
- removed copper zone on In2.Cu, net GND

Commit message: Add labeling silkmask
Other:
- board text added: "+"
- board text added: "+12V"
- board text added: "-"
- board text added: "CK"
- board text added: "DT"
- board text added: "GND"
- board text added: "IN1&2"
- board text added: "IN3"
- board text added: "OUT1"
- board text added: "OUT2"
Changed lines of the file:
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@@
 		(tags "capacitor")
 		(property "Reference" "C7"
-			(at 1.270001 0 360)
+			(at 1.270001 0 0)
 			(layer "F.SilkS")
 			(effects
@@
 		(tags "capacitor")
 		(property "Reference" "C2"
-			(at 0.019146 -0.808222 360)
+			(at 0.019146 -0.808222 0)
 			(layer "F.SilkS")
 			(effects
@@
 		)
 		(property "Value" "100n"
-			(at 0 1.16 360)
+			(at 0 1.16 0)
 			(layer "F.Fab")
 			(effects
@@
 		)
 		(fp_text user "${REFERENCE}"
-			(at 0 0 360)
+			(at 0 0 0)
 			(layer "F.Fab")
 			(effects
@@
 		(tags "capacitor")
 		(property "Reference" "C4"
-			(at -1.3685 -0.028 360)
+			(at -1.3685 -0.028 0)
 			(layer "F.SilkS")
 			(effects
@@
 		)
 		(property "Value" "100n"
-			(at 0 1.16 360)
+			(at 0 1.16 0)
 			(layer "F.Fab")
 			(effects
@@
 		)
 		(fp_text user "${REFERENCE}"
-			(at 0 0 360)
+			(at 0 0 0)
 			(layer "F.Fab")
 			(effects
@@
 		(tags "capacitor")
 		(property "Reference" "C1"
-			(at -1.397 0 360)
+			(at -1.397 0 0)
 			(layer "F.SilkS")
 			(effects
@@
 		)
 		(property "Value" "10u"
-			(at 0 1.16 360)
+			(at 0 1.16 0)
 			(layer "F.Fab")
 			(effects
@@
 		)
 		(fp_text user "${REFERENCE}"
-			(at 0 0 360)
+			(at 0 0 0)
 			(layer "F.Fab")
 			(effects
@@
 		(tags "resistor")
 		(property "Reference" "R4"
-			(at 1.397 0 360)
+			(at 1.397 0 0)
 			(layer "F.SilkS")
 			(effects
@@
 		)
 		(property "Value" "10k"
-			(at 0 1.17 360)
+			(at 0 1.17 0)
 			(layer "F.Fab")
 			(effects
@@
 		)
 		(fp_text user "${REFERENCE}"
-			(at 0 0 360)
+			(at 0 0 0)
 			(layer "F.Fab")
 			(effects
@@
 		(tags "capacitor")
 		(property "Reference" "C9"
-			(at -1.270001 0 360)
+			(at -1.270001 0 0)
 			(layer "F.SilkS")
 			(effects
@@
 		)
 		(property "Value" "AO3400A"
-			(at 0 2.4 360)
+			(at 0 2.4 0)
 			(layer "F.Fab")
 			(effects
@@
 		)
 		(fp_text user "${REFERENCE}"
-			(at 0 0 360)
+			(at 0 0 0)
 			(layer "F.Fab")
 			(effects
@@
 		(tags "SOT TO_SOT_SMD")
 		(property "Reference" "Q1"
-			(at 1.524 1.143 360)
+			(at 1.524 1.143 0)
 			(layer "F.SilkS")
 			(effects
@@
 		(tags "capacitor")
 		(property "Reference" "C5"
-			(at -1.270001 0 360)
+			(at -1.270001 0 0)
 			(layer "F.SilkS")
 			(effects
@@
 		(tags "resistor")
 		(property "Reference" "R1"
-			(at 1.397 0 360)
+			(at 1.397 0 0)
 			(layer "F.SilkS")
 			(effects
@@
 		)
 		(property "Value" "10k"
-			(at 0 1.17 360)
+			(at 0 1.17 0)
 			(layer "F.Fab")
 			(effects
@@
 		)
 		(fp_text user "${REFERENCE}"
-			(at 0 0 360)
+			(at 0 0 0)
 			(layer "F.Fab")
 			(effects
@@
 		(tags "capacitor")
 		(property "Reference" "C3"
-			(at -1.270001 0 360)
+			(at -1.270001 0 0)
 			(layer "F.SilkS")
 			(effects
@@
 		(tags "SMD SMT crystal")
 		(property "Reference" "Y1"
-			(at 2.413 0 360)
+			(at 2.413 0 0)
 			(layer "F.SilkS")
 			(effects
@@
 		(tags "LQFP QFP")
 		(property "Reference" "U2"
-			(at 4.346501 -4.346 360)
+			(at 4.346501 -4.346 0)
 			(layer "F.SilkS")
 			(effects
@@
 		)
 		(property "Value" "STM32F103C8Tx"
-			(at 0 5.85 360)
+			(at 0 5.85 0)
 			(layer "F.Fab")
 			(effects
@@
 		)
 		(fp_text user "${REFERENCE}"
-			(at 0 0 360)
+			(at 0 0 0)
 			(layer "F.Fab")
 			(effects
@@
 		(tags "capacitor")
 		(property "Reference" "C8"
-			(at -0.099 0.888999 360)
+			(at -0.099 0.888999 0)
 			(layer "F.SilkS")
 			(effects
@@
 		)
 		(property "Value" "10p"
-			(at 0 1.16 360)
+			(at 0 1.16 0)
 			(layer "F.Fab")
 			(effects
@@
 		)
 		(fp_text user "${REFERENCE}"
-			(at 0 0 360)
+			(at 0 0 0)
 			(layer "F.Fab")
 			(effects
@@
 		(tags "resistor")
 		(property "Reference" "R12"
-			(at -2.413 -0.381 360)
+			(at -2.413 -0.381 0)
 			(layer "F.SilkS")
 			(effects
@@
 		(tags "resistor")
 		(property "Reference" "R5"
-			(at 1.397 0 360)
+			(at 1.397 0 0)
 			(layer "F.SilkS")
 			(effects
@@
 		(tags "solder jumper open")
 		(property "Reference" "JP1"
-			(at 0 1.8 90)
+			(at 1.808 -2.159 180)
 			(layer "B.SilkS")
 			(effects
@@
 		(tags "tag connect programming header pogo pins")
 		(property "Reference" "J3"
-			(at 4.064 0 360)
+			(at 4.064 0 0)
 			(layer "B.SilkS")
 			(effects
@@
 		(layer "Edge.Cuts")
 	)
+	(gr_text "GND"
+		(at 112.522 63.246 0)
+		(layer "B.SilkS")
+		(effects
+			(font
+				(size 1 1)
+				(thickness 0.2)
+				(bold yes)
+			)
+			(justify left bottom mirror)
+		)
+	)
+	(gr_text "CK"
+		(at 78.994 73.152 0)
+		(layer "B.SilkS")
+		(effects
+			(font
+				(size 1 1)
+				(thickness 0.2)
+				(bold yes)
+			)
+			(justify left bottom mirror)
+		)
+	)
+	(gr_text "+12V"
+		(at 112.522 58.166 0)
+		(layer "B.SilkS")
+		(effects
+			(font
+				(size 1 1)
+				(thickness 0.2)
+				(bold yes)
+			)
+			(justify left bottom mirror)
+		)
+	)
+	(gr_text "OUT2"
+		(at 112.522 73.406 0)
+		(layer "B.SilkS")
+		(effects
+			(font
+				(size 1 1)
+				(thickness 0.2)
+				(bold yes)
+			)
+			(justify left bottom mirror)
+		)
+	)
+	(gr_text "IN3"
+		(at 112.522 78.486 0)
+		(layer "B.SilkS")
+		(effects
+			(font
+				(size 1 1)
+				(thickness 0.2)
+				(bold yes)
+			)
+			(justify left bottom mirror)
+		)
+	)
+	(gr_text "DT"
+		(at 78.994 70.612 0)
+		(layer "B.SilkS")
+		(effects
+			(font
+				(size 1 1)
+				(thickness 0.2)
+				(bold yes)
+			)
+			(justify left bottom mirror)
+		)
+	)
+	(gr_text "IN1&2"
+		(at 116.586 86.106 0)
+		(layer "B.SilkS")
+		(effects
+			(font
+				(size 1 1)
+				(thickness 0.2)
+				(bold yes)
+			)
+			(justify left bottom mirror)
+		)
+	)
+	(gr_text "+"
+		(at 78.232 75.692 0)
+		(layer "B.SilkS")
+		(effects
+			(font
+				(size 1 1)
+				(thickness 0.2)
+				(bold yes)
+			)
+			(justify left bottom mirror)
+		)
+	)
+	(gr_text "OUT1"
+		(at 112.522 68.326 0)
+		(layer "B.SilkS")
+		(effects
+			(font
+				(size 1 1)
+				(thickness 0.2)
+				(bold yes)
+			)
+			(justify left bottom mirror)
+		)
+	)
+	(gr_text "-"
+		(at 78.232 68.072 0)
+		(layer "B.SilkS")
+		(effects
+			(font
+				(size 1 1)
+				(thickness 0.2)
+				(bold yes)
+			)
+			(justify left bottom mirror)
+		)
+	)
 	(segment

Commit message: Make production files
Parts:
- removed D4: MM1Z3V3, Diode_SMD:D_SOD-123
- removed J5: Conn_01x04_Pin, Connector_PinHeader_2.54mm:PinHeader_1x04_P2.54mm_Vertical
- removed R15: 18k, Resistor_SMD:R_1206_3216Metric
- removed R16: 2k2, Resistor_SMD:R_1206_3216Metric
- added C19: 10n, Capacitor_SMD:C_0402_1005Metric, F.Cu at (96.4, 70.6)
- added C20: 1u, Capacitor_SMD:C_0402_1005Metric, F.Cu at (97.4, 70.6)
- added C21: 1u, Capacitor_SMD:C_0402_1005Metric, F.Cu at (97.4, 73.0)
- added C22: 47u, Capacitor_SMD:C_1206_3216Metric, F.Cu at (79.0, 69.9)
- added D5: SS54, Diode_SMD:D_SMA, F.Cu at (104.4, 78.1)
- added FB1: 100, Inductor_SMD:L_0805_2012Metric, F.Cu at (99.5, 72.2)
- added R20: 10k, Resistor_SMD:R_0402_1005Metric, F.Cu at (102.0, 80.6)
- added R21: 5k1, Resistor_SMD:R_0402_1005Metric, F.Cu at (100.9, 80.6)
- added R22: 47k, Resistor_SMD:R_0402_1005Metric, F.Cu at (99.3, 80.1)
- added R23: 12k, Resistor_SMD:R_0402_1005Metric, F.Cu at (99.3, 81.2)
- added U5: SSD1306, User_Footprints:SSD1309_1.3, F.Cu at (92.7, 49.8)
- J4: footprint TerminalBlock:TerminalBlock_bornier-6_P5.08mm -> User_Footprints:ScrewTerminalPlug_6P_P5.08
- R14, R19: value 4k7 -> 5k1
- U2: value STM32F103C8Tx -> STM32G431CBTx
- moved G1 31.8 mm to (94.5, 54.6)
- moved J4 12.8 mm to (113.3, 70.1), turned to 0 degrees
- moved C2 11.9 mm to (96.3, 68.5), turned to -90 degrees
- moved C3 10.9 mm to (87.7, 65.6), turned to 0 degrees
- moved Y1 10.2 mm to (88.4, 79.5), turned to 180 degrees
- moved C8 10.2 mm to (91.1, 80.3), turned to 90 degrees
- moved R4 9.40 mm to (84.8, 73.3), turned to 90 degrees
- moved C7 8.84 mm to (92.1, 80.3), turned to -90 degrees
- moved C9 8.59 mm to (87.3, 77.2), turned to 0 degrees
- moved C4 7.08 mm to (85.3, 75.2), turned to 180 degrees
- moved R8 6.92 mm to (91.7, 61.1), turned to 180 degrees
- moved R5 6.88 mm to (89.2, 77.2), turned to 0 degrees
- moved R14 6.36 mm to (107.5, 77.0), turned to 0 degrees
- moved R13 5.42 mm to (107.5, 78.1), turned to 180 degrees
- moved R9 5.21 mm to (89.5, 61.1), turned to 0 degrees
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Connections:
- J4 pad 5: /SNS3 -> /SNS1
- JP1 pad 1: /SNS2 -> /SNST
- JP1 pad 3: /SNS1 -> /SNS2
- R12 pad 2: /SNS3 -> /SNS1
- R13 pad 1: /SNS3 -> /SNS1
- R13 pad 2: /SIG3 -> /SIG1
- R14 pad 1: /SIG3 -> /SIG1
- U2 pad 11: unconnected-(U2-PA1-Pad11) -> /SIG1
- U2 pad 13: /SIG2 -> /BTN3
- U2 pad 14: /SIG3 -> unconnected-(U2-PA6-Pad14)
- U2 pad 15: /SIG1 -> unconnected-(U2-PA7-Pad15)
- U2 pad 16: /DRV2 -> /TACH
- U2 pad 17: /DRV1 -> unconnected-(U2-PB1-Pad17)
- U2 pad 18: unconnected-(U2-PB0-Pad18) -> /BTN4
- U2 pad 19: unconnected-(U2-PB1-Pad19) -> GND
- U2 pad 2: unconnected-(U2-PC13-Pad2) -> /BTN1
- U2 pad 20: unconnected-(U2-PB2-Pad20) -> +3V3A
- U2 pad 21: /SCLD -> +3V3A
- U2 pad 22: /SDAD -> unconnected-(U2-PB10-Pad22)
- U2 pad 25: /PGPS -> /DRV2
- U2 pad 26: unconnected-(U2-PB13-Pad26) -> /DRV1
- U2 pad 3: /BTN3 -> unconnected-(U2-PC14-Pad3)
- U2 pad 30: /GPS_TX -> /SDAD
- U2 pad 31: /GPS_RX -> /SCLD
- U2 pad 33: unconnected-(U2-PA12-Pad33) -> /PGPS
- U2 pad 34: /SWDIO -> unconnected-(U2-PA12-Pad34)
- U2 pad 37: /SWCLK -> /SWDIO
- U2 pad 38: unconnected-(U2-PA15-Pad38) -> /SWCLK
- U2 pad 39: /SWO -> /SCLE
- U2 pad 4: /BTN4 -> unconnected-(U2-PC15-Pad4)
- U2 pad 40: unconnected-(U2-PB4-Pad40) -> /SWO
- U2 pad 42: /SCLE -> /BTN2
- U2 pad 43: /SDAE -> /GPS_TX
- U2 pad 44: /BOOT0 -> /GPS_RX
- U2 pad 45: /BTN1 -> /BOOT0
- U2 pad 46: /BTN2 -> /SDAE
- U2 pad 8: GND -> /TACH
- U2 pad 9: +3V3 -> /SIG2
Routing:
- net /SIG3: track 19.2 -> 0.00 mm
- net /SNS3: track 17.7 -> 0.00 mm, vias 1 -> 0
- net /TACH: track 0.00 -> 16.8 mm
- net /SNST: track 0.00 -> 13.7 mm, vias 0 -> 1
- net /SWO: track 30.7 -> 18.2 mm
- net /SIG2: track 26.2 -> 18.3 mm, vias 0 -> 2
- net /SNS1: track 13.4 -> 5.55 mm, vias 1 -> 0
- net /SIG1: track 23.7 -> 16.9 mm
- net Net-(Q1-D): track 13.7 -> 7.34 mm, vias 0 -> 2
- net +3V3A: track 0.00 -> 5.67 mm
- net /BTN2: track 17.8 -> 23.3 mm
- net /SWCLK: track 33.0 -> 27.7 mm
- net /SDAD: track 24.4 -> 19.7 mm
- net /Tac1/PROT: track 0.00 -> 4.60 mm
- net +12V: track 65.7 -> 70.1 mm
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Other:
- board text added: "3V3"
- board text added: "S2"
- board text added: "SCL"
- board text added: "SDA"
- board text added: "SNS1"
- board text added: "SNS2/TACH"
- board text added: "T"
- board text removed: "IN1&2"
- board text removed: "IN3"

Commit message: Fix power connection
Parts:
- removed Q1: AO3400A, Package_TO_SOT_SMD:SOT-23
- removed Q2: AO3401A, Package_TO_SOT_SMD:SOT-23
- removed R1: 10k, Resistor_SMD:R_0402_1005Metric
- Q3, Q5: value Q_Dual_PMOS_S1G1S2G2D2D2D1D1 -> DMP4025LSD-VB
Connections:
- C22 pad 1: Net-(J1-Pin_1) -> +5V
- J1 pad 1: Net-(J1-Pin_1) -> +5V
- U2 pad 33: /PGPS -> unconnected-(U2-PA11-Pad33)
Routing:
- net +5V: track 19.4 -> 35.9 mm
- net /PGPS: track 8.32 -> 0.00 mm
- net Net-(Q1-D): track 7.34 -> 0.00 mm, vias 2 -> 0
- net Net-(J1-Pin_1): track 7.12 -> 0.00 mm
- net +3V3: track 61.7 -> 56.5 mm
- net GND: track 100.0 -> 99.0 mm, vias 30 -> 29
